Commit message: Fix TF tree: adjust LDS-M300-E scan_joint origin and remove redundant base_footprint_to_base_link static tf. Add cmd_vel watchdog to robot_control

File: src/omorobot/omorobot_description/urdf/DONKEYBOTI.urdf (robot description, URDF)
Before this commit: robot DONKEYBOTI, 6 links, 5 joints
Joints:
- joint scan_joint: origin xyz=-0.335 0.0 0.432 rpy=0.0 0.0 0.0 -> xyz=0.335 0.0 0.5295 rpy=0.0 0.0 0.0
